File: Hardware/2D_PCB.brd (EAGLE design)
At the start: 46 x 35 mm, 105 parts, among them IC1 BQ25180YBGR, IC2 DRV2605YZFR, IC3 BMA421, IC9 RT6160AWSC, J1 503480-2400_503480-2400, J2 TC2030-IDC, J4 KH-TYPE-C-16P, Q3 SI1308EDL-T1-GE3, U1 NRF52840_QF, U3 MAX17048G+T10, X1 32MHz, X2 32.768kHz

Commit message: Added Project Second Iteration
Parts:
- moved J4 2.84 mm to (-0.87, 16.5)
- moved U3 2.72 mm to (-8.00, 14.9)
- moved C27 1.65 mm to (-16.7, 13.1)
- moved IC2 1.53 mm to (-12.8, 11.0)
- moved TP_OP 1.48 mm to (-13.3, 15.1)
- moved C43 1.47 mm to (-2.49, 9.40)
- moved TP_ON 1.38 mm to (-15.5, 14.7)
- moved TP_VBAT 1.14 mm to (-19.0, 15.5)
- moved TP_VBAT_GND 1.02 mm to (-18.9, 11.7)
- moved C32 0.96 mm to (-11.7, 12.8)
- moved R18 0.33 mm to (12.1, 14.9)
- moved TP_VREG 0.33 mm to (2.36, 1.30)
- moved TP_GND 0.16 mm to (15.2, -5.19)
- moved R9 0.15 mm to (16.6, 14.5)
- moved EPD_C2 0.10 mm to (-11.7, 0.03)
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Routing:
- net GND: track 267.8 -> 274.6 mm
- net DP: track 10.8 -> 15.5 mm
- net VBAT/1.2A: track 23.5 -> 19.2 mm
- net VBUS/1.5D: track 72.9 -> 76.8 mm
- net 3V3/2.4A: track 131.0 -> 134.7 mm, vias 10 -> 12
- net DN: track 10.2 -> 13.8 mm
- net RF: track 24.9 -> 28.0 mm
- net SDA/1.4C: track 9.02 -> 6.29 mm
- net OUT+: track 13.2 -> 10.8 mm
- net N$18: track 2.91 -> 4.67 mm
- net SCL/1.4C: track 7.87 -> 6.32 mm
- net OUT-: track 12.0 -> 13.5 mm
- net VREG: track 42.5 -> 43.9 mm
- net 3V3/1.7D: track 53.7 -> 55.1 mm
- net VBUS/2.6D: track 26.1 -> 27.4 mm
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