File: Hardware/Schematic.sch (EAGLE design)
At the start: 105 parts, among them IC1 BQ25180YBGR, IC2 DRV2605YZFR, IC3 BMA421, IC9 RT6160AWSC, J1 503480-2400_503480-2400, J2 TC2030-IDC, J4 KH-TYPE-C-16P, Q3 SI1308EDL-T1-GE3, U1 NRF52840_QF, U3 MAX17048G+T10, X1 32MHz, X2 32.768kHz

Commit message: Added Project Second Iteration
Other:
- note removed: "Cernea Mihnea-Ioan"
